File: Diseño PCB/KiCAD/Asocontador_PCB/Asocontador_PCB.kicad_pcb (KiCad board)
At the start: 2 copper layers, 101.6 x 76.2 mm, 2 parts

Commit message: Modificaciones Varias
Parts:
- added 4-20mA-5v1: Conn_01x03_Socket, Connector_JST:JST_EH_B3B-EH-A_1x03_P2.50mm_Vertical, F.Cu at (156.8, 108.7)
- added C1: 220uF_25V, Capacitor_THT:CP_Radial_D8.0mm_P3.50mm, F.Cu at (99.6, 89.2)
- added DS1: WC1602A, Display:WC1602A, F.Cu at (108.7, 45.7)
- added J1: Screw_Terminal_2_P5.00mm, TerminalBlock_Phoenix:TerminalBlock_Phoenix_PT-1,5-2-5.0-H_1x02_P5.00mm_Horizontal, F.Cu at (99.1, 108.2)
- added R1: 220, Resistor_THT:R_Axial_DIN0207_L6.3mm_D2.5mm_P10.16mm_Horizontal, F.Cu at (185.4, 50.5)
- added REF**: MountingHole_2.2mm_M2_ISO7380_Pad, MountingHole:MountingHole_2.2mm_M2_ISO7380_Pad, F.Cu at (96.5, 45.7)
- added REF**: MountingHole_2.2mm_M2_ISO7380_Pad, MountingHole:MountingHole_2.2mm_M2_ISO7380_Pad, F.Cu at (137.2, 109.2)
- added REF**: MountingHole_2.2mm_M2_ISO7380_Pad, MountingHole:MountingHole_2.2mm_M2_ISO7380_Pad, F.Cu at (188.0, 45.7)
- added RV1: potentiometer_RM065, PCM_SL_Devices:Potentiometer_RM065, F.Cu at (185.5, 66.8)
- added Turbidez1: Conn_01x03_Socket, Connector_JST:JST_EH_B3B-EH-A_1x03_P2.50mm_Vertical, F.Cu at (180.2, 108.7)
- added U1: LM7805_TO220, Package_TO_SOT_THT:TO-220F-3_Horizontal_TabDown, F.Cu at (113.3, 103.4)
- added pH1: Conn_01x03_Socket, Connector_JST:JST_EH_B3B-EH-A_1x03_P2.50mm_Vertical, F.Cu at (168.5, 108.7)
- moved D1 69.2 mm to (106.7, 99.1), turned to 180 degrees
- moved Arduino1 8.02 mm to (148.3, 98.8)
- renumbered A1 to Arduino1
Connections:
- Arduino1 pad 27: unconnected-(A1-+5V-Pad27) -> Net-(Arduino1-+5V)
- Arduino1 pad 5: unconnected-(A1-D2-Pad5) -> Net-(Arduino1-D2)
- Arduino1 pad 6: unconnected-(A1-D3-Pad6) -> Net-(Arduino1-D3)
Routing:
- net GND: track 0.00 -> 34.0 mm
- net Net-(D1-K): track 0.00 -> 31.0 mm
- net Net-(D1-A): track 0.00 -> 10.2 mm
