File: Diseño PCB/KiCAD/Asocontador_PCB/Asocontador_PCB.kicad_pcb (KiCad board)
At the start: 2 copper layers, 101.6 x 76.2 mm, 14 parts, among them J1 Screw_Terminal_2_P5.00mm, U1 LM7805_TO220

Commit message: Cambios varios
Parts:
- added D2: LED, LED_THT:LED_D3.0mm, F.Cu at (125.6, 87.5)
- added D3: LED, LED_THT:LED_D3.0mm, F.Cu at (130.5, 87.5)
- added R2: 220, Resistor_THT:R_Axial_DIN0207_L6.3mm_D2.5mm_P10.16mm_Horizontal, F.Cu at (123.9, 93.2)
- added R3: 220, Resistor_THT:R_Axial_DIN0207_L6.3mm_D2.5mm_P10.16mm_Horizontal, F.Cu at (123.9, 97.8)
- moved R1 50.9 mm to (145.9, 82.7), turned to 0 degrees
- moved Arduino1 3.62 mm to (148.5, 102.4)
- moved RV1 0.88 mm to (186.0, 76.0)
Connections:
- net Net-(Arduino1-D2) renamed D2
- net Net-(Arduino1-VIN) renamed VIN
- 4-20mA-5v1 pad 1: unconnected-(4-20mA-5v1-Pin_1-Pad1) -> A1
- 4-20mA-5v1 pad 2: unconnected-(4-20mA-5v1-Pin_2-Pad2) -> +5V
- 4-20mA-5v1 pad 3: unconnected-(4-20mA-5v1-Pin_3-Pad3) -> GND
- Arduino1 pad 1: unconnected-(Arduino1-D1/TX-Pad1) -> D1
- Arduino1 pad 10: unconnected-(Arduino1-D7-Pad10) -> D7
- Arduino1 pad 11: unconnected-(Arduino1-D8-Pad11) -> D8
- Arduino1 pad 12: unconnected-(Arduino1-D9-Pad12) -> D9
- Arduino1 pad 13: unconnected-(Arduino1-D10-Pad13) -> D10
- Arduino1 pad 14: unconnected-(Arduino1-D11-Pad14) -> D11
- Arduino1 pad 15: unconnected-(Arduino1-D12-Pad15) -> D12
- Arduino1 pad 16: unconnected-(Arduino1-D13-Pad16) -> D13
- Arduino1 pad 17: unconnected-(Arduino1-3V3-Pad17) -> 3V3
- Arduino1 pad 19: unconnected-(Arduino1-A0-Pad19) -> A0
- Arduino1 pad 2: unconnected-(Arduino1-D0/RX-Pad2) -> D0
- Arduino1 pad 20: unconnected-(Arduino1-A1-Pad20) -> A1
- Arduino1 pad 21: unconnected-(Arduino1-A2-Pad21) -> A2
- Arduino1 pad 22: unconnected-(Arduino1-A3-Pad22) -> A3
- Arduino1 pad 23: unconnected-(Arduino1-A4-Pad23) -> A4
- Arduino1 pad 24: unconnected-(Arduino1-A5-Pad24) -> A5
- Arduino1 pad 25: unconnected-(Arduino1-A6-Pad25) -> A6
- Arduino1 pad 26: unconnected-(Arduino1-A7-Pad26) -> A7
- Arduino1 pad 6: Net-(Arduino1-D3) -> D3
- Arduino1 pad 7: unconnected-(Arduino1-D4-Pad7) -> D4
- Arduino1 pad 8: unconnected-(Arduino1-D5-Pad8) -> D5
- Arduino1 pad 9: unconnected-(Arduino1-D6-Pad9) -> D6
- DS1 pad 11: unconnected-(DS1-D4-Pad11) -> D4
- DS1 pad 12: unconnected-(DS1-D5-Pad12) -> D5
- DS1 pad 13: unconnected-(DS1-D6-Pad13) -> D6
- DS1 pad 14: unconnected-(DS1-D7-Pad14) -> D7
- DS1 pad 2: Net-(DS1-VDD) -> +5V
- DS1 pad 4: unconnected-(DS1-RS-Pad4) -> D3
- DS1 pad 5: Net-(Arduino1-D3) -> GND
- RV1 pad 1: Net-(DS1-VDD) -> +5V
- Turbidez1 pad 1: unconnected-(Turbidez1-Pin_1-Pad1) -> A2
- Turbidez1 pad 2: unconnected-(Turbidez1-Pin_2-Pad2) -> +5V
- Turbidez1 pad 3: unconnected-(Turbidez1-Pin_3-Pad3) -> GND
- pH1 pad 1: unconnected-(pH1-Pin_1-Pad1) -> A0
- pH1 pad 2: unconnected-(pH1-Pin_2-Pad2) -> +5V
- pH1 pad 3: unconnected-(pH1-Pin_3-Pad3) -> GND
Routing:
- net Net-(Arduino1-D3): track 193.2 -> 0.00 mm
- net +5V: track 0.00 -> 191.2 mm
- net (no net): track 110.0 -> 0.00 mm
- net D3: track 0.00 -> 98.2 mm
- net D7: track 0.00 -> 84.6 mm
- net D6: track 0.00 -> 83.3 mm
- net D5: track 0.00 -> 81.3 mm
- net D4: track 0.00 -> 80.5 mm
- net D2: track 188.3 -> 117.5 mm, vias 0 -> 4
- net A1: track 0.00 -> 54.5 mm
- net D9: track 0.00 -> 48.6 mm, vias 0 -> 1
- net D8: track 0.00 -> 44.9 mm, vias 0 -> 1
- net A0: track 0.00 -> 43.4 mm
- net A2: track 0.00 -> 41.1 mm
- net GND: track 332.9 -> 370.5 mm
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