File: Diseño PCB/KiCAD/Asocontador_PCB/Asocontador_PCB.kicad_pcb (KiCad board)
At the start: 2 copper layers, 101.6 x 76.2 mm, 18 parts, among them J1 Screw_Terminal_2_P5.00mm, U1 LM7805_TO220

Commit message: cAMBIOS
Routing:
- net GND: track 370.5 -> 364.6 mm
Changed lines of the file:
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@@
     (fp_arc (start 63.7 8) (mid 64.053553 8.146447) (end 64.2 8.5)
       (stroke (width 0.12) (type solid)) (layer "F.SilkS"))
-    (fp_arc (start 64.20104 22.49932) (mid 64.054479 22.85315) (end 63.70066 22.9997)
+    (fp_arc (start 64.20104 22.49932) (mid 64.054473 22.853115) (end 63.70066 22.9997)
       (stroke (width 0.12) (type solid)) (layer "F.SilkS"))
     (fp_line (start -8.25 -2.75) (end -8.25 33.75)
@@
     (stroke (width 0.1) (type default)) (fill none) (layer "Edge.Cuts"))
   (segment (start 146.812 45.72) (end 146.812 74.982) (width 0.5) (layer "F.Cu") (net 1))
-  (segment (start 156.12 102.42) (end 156.12 104.39) (width 0.5) (layer "F.Cu") (net 1))
   (segment (start 108.712 45.72) (end 108.712 44.228) (width 0.5) (layer "F.Cu") (net 1))
   (segment (start 146.812 74.982) (end 151.17 79.34) (width 0.5) (layer "F.Cu") (net 1))
@@
   (segment (start 108.712 44.228) (end 109.86 43.08) (width 0.5) (layer "F.Cu") (net 1))
   (segment (start 96.61 63.88) (end 108.72 51.77) (width 0.5) (layer "F.Cu") (net 1))
-  (segment (start 156.12 104.39) (end 156 104.51) (width 0.5) (layer "F.Cu") (net 1))
   (segment (start 100.49 94.69) (end 97.47 94.69) (width 0.5) (layer "F.Cu") (net 1))
   (segment (start 108.72 51.77) (end 108.712 51.762) (width 0.5) (layer "F.Cu") (net 1))
   (segment (start 151.17 79.34) (end 179.98 79.34) (width 0.5) (layer "F.Cu") (net 1))
   (segment (start 96.61 93.83) (end 96.61 63.88) (width 0.5) (layer "F.Cu") (net 1))
-  (segment (start 154.56 105.95) (end 152.85 105.95) (width 0.5) (layer "F.Cu") (net 1))
   (segment (start 108.712 51.762) (end 108.712 45.72) (width 0.5) (layer "F.Cu") (net 1))
   (segment (start 97.47 94.69) (end 96.61 93.83) (width 0.5) (layer "F.Cu") (net 1))
@@
   (segment (start 118.89 43.37) (end 118.872 43.388) (width 0.5) (layer "F.Cu") (net 1))
   (segment (start 109.86 43.08) (end 118.6 43.08) (width 0.5) (layer "F.Cu") (net 1))
-  (segment (start 156 104.51) (end 154.56 105.95) (width 0.5) (layer "F.Cu") (net 1))
   (segment (start 125.57 85.41) (end 126.68 84.3) (width 0.5) (layer "B.Cu") (net 1))
   (segment (start 131.9 84.5) (end 150.57 84.5) (width 0.5) (layer "B.Cu") (net 1))
