File: Diseño PCB/KiCAD/Asocontador_PCB/_autosave-Asocontador_PCB.kicad_pcb (KiCad board)
At the start: 2 copper layers, 101.6 x 76.2 mm, 14 parts, among them J1 Screw_Terminal_2_P5.00mm, U1 LM7805_TO220

Commit message: Modificaciones varias
Parts:
- moved R1 8.51 mm to (185.1, 59.0)
Routing:
- net Net-(DS1-VDD): track 0.00 -> 105.6 mm
- net GND: track 332.9 -> 391.5 mm
- net +5V: track 0.00 -> 42.4 mm
- net Net-(DS1-LED(+)): track 50.0 -> 56.9 mm
Changed lines of the file:
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@@
   )
   (footprint "Resistor_THT:R_Axial_DIN0207_L6.3mm_D2.5mm_P10.16mm_Horizontal" (layer "F.Cu")
-    (at 185.42 50.546 -90)
+    (at 185.13 59.05 -90)
     (descr "Resistor, Axial_DIN0207 series, Axial, Horizontal, pin pitch=10.16mm, 0.25W = 1/4W, length*diameter=6.3*2.5mm^2, http://cdn-reichelt.de/documents/datenblatt/B400/1_4W%23YAG.pdf")
     (tags "Resistor Axial_DIN0207 series Axial Horizontal pin pitch 10.16mm 0.25W = 1/4W length 6.3mm diameter 2.5mm")
@@
   (segment (start 153.51 78.84) (end 134.59 78.84) (width 0.5) (layer "B.Cu") (net 0))
   (segment (start 187.66 86.56) (end 187.66 78) (width 0.5) (layer "B.Cu") (net 0))
+  (segment (start 182.66 79.92) (end 183.57 80.83) (width 0.5) (layer "F.Cu") (net 1))
+  (segment (start 188.39 80.83) (end 189.08 81.52) (width 0.5) (layer "F.Cu") (net 1))
+  (segment (start 182.66 78) (end 182.66 79.92) (width 0.5) (layer "F.Cu") (net 1))
+  (segment (start 189.08 81.52) (end 189.08 94.14) (width 0.5) (layer "F.Cu") (net 1))
+  (segment (start 155.956 95.544) (end 155.956 98.806) (width 0.5) (layer "F.Cu") (net 1))
+  (segment (start 188.92 94.3) (end 157.2 94.3) (width 0.5) (layer "F.Cu") (net 1))
+  (segment (start 183.57 80.83) (end 188.39 80.83) (width 0.5) (layer "F.Cu") (net 1))
+  (segment (start 157.2 94.3) (end 155.956 95.544) (width 0.5) (layer "F.Cu") (net 1))
+  (segment (start 189.08 94.14) (end 188.92 94.3) (width 0.5) (layer "F.Cu") (net 1))
   (segment (start 150.876 81.056) (end 150.35 80.53) (width 0.5) (layer "B.Cu") (net 1))
   (segment (start 97.86 91.77) (end 97.86 86.93) (width 0.5) (layer "B.Cu") (net 1))
@@
   (segment (start 105.07 87.29) (end 106.68 88.9) (width 0.5) (layer "B.Cu") (net 2))
   (segment (start 100.15 87.29) (end 105.07 87.29) (width 0.5) (layer "B.Cu") (net 2))
-  (segment (start 185.166 50.8) (end 184.912 50.546) (width 0.5) (layer "B.Cu") (net 12))
+  (segment (start 155.956 71.256) (end 155.956 83.566) (width 0.5) (layer "F.Cu") (net 11))
+  (segment (start 157.95 69.21) (end 155.93 71.23) (width 0.5) (layer "F.Cu") (net 11))
+  (segment (start 155.93 71.23) (end 155.956 71.256) (width 0.5) (layer "F.Cu") (net 11))
+  (segment (start 185.13 69.21) (end 157.95 69.21) (width 0.5) (layer "F.Cu") (net 11))
   (segment (start 172.72 53.34) (end 175.514 50.546) (width 0.5) (layer "B.Cu") (net 12))
-  (segment (start 175.514 50.546) (end 185.42 50.546) (width 0.5) (layer "B.Cu") (net 12))
+  (segment (start 185.13 59.05) (end 185.13 52.236) (width 0.5) (layer "B.Cu") (net 12))
   (segment (start 144.272 52.832) (end 144.78 53.34) (width 0.5) (layer "B.Cu") (net 12))
+  (segment (start 185.13 52.236) (end 183.44 50.546) (width 0.5) (layer "B.Cu") (net 12))
   (segment (start 144.78 53.34) (end 172.72 53.34) (width 0.5) (layer "B.Cu") (net 12))
   (segment (start 144.272 45.72) (end 144.272 52.832) (width 0.5) (layer "B.Cu") (net 12))
-  (segment (start 187.35 67.2) (end 136.61 67.2) (width 0.5) (layer "B.Cu") (net 18))
+  (segment (start 175.514 50.546) (end 183.44 50.546) (width 0.5) (layer "B.Cu") (net 12))
+  (segment (start 187.66 53.05) (end 185.71 51.1) (width 0.5) (layer "F.Cu") (net 13))
+  (segment (start 185.71 51.1) (end 114.602 51.1) (width 0.5) (layer "F.Cu") (net 13))
+  (segment (start 114.602 51.1) (end 111.252 47.75) (width 0.5) (layer "F.Cu") (net 13))
+  (segment (start 187.66 78) (end 187.66 53.05) (width 0.5) (layer "F.Cu") (net 13))
+  (segment (start 111.252 47.75) (end 111.252 45.72) (width 0.5) (layer "F.Cu") (net 13))
   (segment (start 189.59 90.85) (end 189.59 90.78) (width 0.25) (layer "B.Cu") (net 18))
   (segment (start 158.496 102.044) (end 157.07 103.47) (width 0.5) (layer "B.Cu") (net 18))
+  (segment (start 190.72 70.57) (end 186.86 66.71) (width 0.5) (layer "B.Cu") (net 18))
+  (segment (start 141.37 103.47) (end 139.04 101.14) (width 0.5) (layer "B.Cu") (net 18))
   (segment (start 190.72 89.65) (end 190.72 70.57) (width 0.5) (layer "B.Cu") (net 18))
-  (segment (start 141.37 103.47) (end 139.04 101.14) (width 0.5) (layer "B.Cu") (net 18))
   (segment (start 158.496 98.806) (end 158.496 102.044) (width 0.5) (layer "B.Cu") (net 18))
   (segment (start 157.07 103.47) (end 141.37 103.47) (width 0.5) (layer "B.Cu") (net 18))
+  (segment (start 186.86 66.71) (end 136.12 66.71) (width 0.5) (layer "B.Cu") (net 18))
   (segment (start 140.37 90.85) (end 189.59 90.85) (width 0.5) (layer "B.Cu") (net 18))
+  (segment (start 139.04 92.18) (end 140.37 90.85) (width 0.5) (layer "B.Cu") (net 18))
   (segment (start 189.59 90.78) (end 190.72 89.65) (width 0.5) (layer "B.Cu") (net 18))
-  (segment (start 139.04 92.18) (end 140.37 90.85) (width 0.5) (layer "B.Cu") (net 18))
   (segment (start 139.04 101.14) (end 139.04 92.18) (width 0.5) (layer "B.Cu") (net 18))
-  (segment (start 136.61 67.2) (end 121.412 52.002) (width 0.5) (layer "B.Cu") (net 18))
   (segment (start 121.412 52.002) (end 121.412 45.72) (width 0.5) (layer "B.Cu") (net 18))
-  (segment (start 190.72 70.57) (end 187.35 67.2) (width 0.5) (layer "B.Cu") (net 18))
+  (segment (start 136.12 66.71) (end 121.412 52.002) (width 0.5) (layer "B.Cu") (net 18))
   (segment (start 139.85 89.64) (end 188.12 89.64) (width 0.5) (layer "B.Cu") (net 19))
   (segment (start 137.8 91.69) (end 139.85 89.64) (width 0.5) (layer "B.Cu") (net 19))
