File: Diseño PCB/KiCAD/Asocontador_PCB/Asocontador_PCB.kicad_sch (KiCad schematic)
At the start: 4 parts, among them U2 LM7805_TO220

Commit message: Modificaciones Varias
Parts:
- removed U2: LM7805_TO220, Package_TO_SOT_THT:TO-220-3_Vertical, symbol Regulator_Linear:LM7805_TO220
- added 4-20mA-5v1, Turbidez1, pH1: Conn_01x03_Socket, Connector_JST:JST_EH_B3B-EH-A_1x03_P2.50mm_Vertical, symbol Connector:Conn_01x03_Socket
- added C1: 220uF_25V, Capacitor_THT:CP_Radial_D8.0mm_P3.50mm, symbol PCM_SL_Capacitors:220uF_25V
- added J1: Screw_Terminal_2_P5.00mm, TerminalBlock_Phoenix:TerminalBlock_Phoenix_PT-1,5-2-5.0-H_1x02_P5.00mm_Horizontal, symbol PCM_SL_Screw_Terminal:Screw_Terminal_2_P5.00mm
- added R1: 220, Resistor_THT:R_Axial_DIN0207_L6.3mm_D2.5mm_P10.16mm_Horizontal, symbol PCM_SL_Devices:Resistor
- added RV1: potentiometer_RM065, PCM_SL_Devices:Potentiometer_RM065, symbol PCM_SL_Devices:potentiometer_RM065
- added U1: LM7805_TO220, Package_TO_SOT_THT:TO-220F-3_Horizontal_TabDown, symbol Regulator_Linear:LM7805_TO220
- renumbered A1 to Arduino1
Connections:
- net GND: now also C1.2, J1.2, RV1.3, U1.2 (GND)
- net at D1.1 (K): now also C1.1, U1.1 (VI)
- net at Arduino1.30 (VIN): now also U1.3 (VO)
- net at D1.2 (A): now also J1.1
- net at DS1.15 (LED(+)): now also R1.1
- net at Arduino1.27 (+5V), DS1.2 (VDD): now also RV1.1
- net VO: now reaches DS1.3 (VO)
- net VO: now also RV1.2
- net at DS1.4 (RS): no longer Arduino1.7 (D4)
Other:
- company: (none) -> Tecnoparque Nodo Pitalito
- title: (none) -> Esquemático Asocontador
- moved on the sheet: D1

Commit message: Modificaciones varias
Connections:
- net GND: now also DS1.16 (LED(-))
- net VIN: now reaches Arduino1.30 (VIN), U1.3 (VO)
- net +5V: now reaches Arduino1.27 (+5V), DS1.2 (VDD), RV1.1
- net +5V: now also R1.2
- net at DS1.5 (R/W): no longer Arduino1.6 (D3)
- net at DS1.6 (E): no longer Arduino1.5 (D2)
- net D1: now reaches Arduino1.1 (D1/TX)
- net D7: now reaches Arduino1.10 (D7)
- net D8: now reaches Arduino1.11 (D8)
- net D9: now reaches Arduino1.12 (D9)
- net D10: now reaches Arduino1.13 (D10)
- net D11: now reaches Arduino1.14 (D11)
- net D12: now reaches Arduino1.15 (D12)
- net D13: now reaches Arduino1.16 (D13)
- net 3V3: now reaches Arduino1.17 (3V3)
- net A0: now reaches Arduino1.19 (A0)
- net D0: now reaches Arduino1.2 (D0/RX)
- net A1: now reaches Arduino1.20 (A1)
- net A2: now reaches Arduino1.21 (A2)
- net A3: now reaches Arduino1.22 (A3)
- net A4: now reaches Arduino1.23 (A4)
- net A5: now reaches Arduino1.24 (A5)
- net A6: now reaches Arduino1.25 (A6)
- net A7: now reaches Arduino1.26 (A7)
- net D4: now reaches Arduino1.7 (D4)
- net D5: now reaches Arduino1.8 (D5)
- net D6: now reaches Arduino1.9 (D6)
- new net D2: Arduino1.5 (D2)
- new net D3: Arduino1.6 (D3)
Other:
- note added: "Etapa de Alimentación"
- note added: "Etapa de Control"
- note added: "Etapa de Visualización"
- moved on the sheet: 4-20mA-5v1, Arduino1, C1, D1, DS1, J1, R1, RV1, Turbidez1, U1, pH1

Commit message: Cambios varios
Parts:
- added D2, D3: LED, LED_THT:LED_D3.0mm, symbol Device:LED
- added R2, R3: 220, Resistor_THT:R_Axial_DIN0207_L6.3mm_D2.5mm_P10.16mm_Horizontal, symbol PCM_SL_Devices:Resistor
Connections:
- net +5V: now also 4-20mA-5v1.2 (Pin_2), Turbidez1.2 (Pin_2), pH1.2 (Pin_2)
- net A0: now also pH1.1 (Pin_1)
- net A1: now also 4-20mA-5v1.1 (Pin_1)
- net A2: now also Turbidez1.1 (Pin_1)
- net D2: now also DS1.6 (E)
- net D3: now also DS1.4 (RS)
- net D4: now also DS1.11 (D4)
- net D5: now also DS1.12 (D5)
- net D6: now also DS1.13 (D6)
- net D7: now also DS1.14 (D7)
- net D8: now also R2.2
- net D9: now also R3.2
- net GND: now also 4-20mA-5v1.3 (Pin_3), DS1.5 (R/W), Turbidez1.3 (Pin_3), pH1.3 (Pin_3), D2.1 (K), D3.1 (K)
- new net: D3.2 (A), R3.1
- new net: D2.2 (A), R2.1
- no-connect marks 0 -> 4
Other:
- note added: "Etapa de Sensores"
- moved on the sheet: 4-20mA-5v1, Turbidez1, pH1
